File: Uno.kicad_pcb (KiCad board)
At the start: 2 copper layers, 68.5 x 53.3 mm, 73 parts, among them J1 JTAG, J2 POWER, J3 ANALOG, J4 ICSP, J5 Conn_01x08, J6 DIGITAL-HIGH, J7 DIGITAL-LOW, J8 USB_B, J9 PJ-202A, Q1 2N7002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

Commit message: Move to KiCAD 5.99 and release v1.0.0
Other:
- net class Default removed
- rule pad_to_mask_clearance: 0.05 -> 0
- board text added: "v1.0.0"
